File: 411 Project/nocLock/100-Schematics/nocLock.sch (EAGLE design)
At the start: 2 parts, among them U1 ATMEGA328

Commit message: Added lib and edited BOM
Parts:
- removed IC1: (no value), v-reg:78XXL
- added C1: 100nF, rcl:C-USC0805K
- added C2, C3, C4, C5: (no value), rcl:C-USC0805K
- added L1: 100uH, rcl:L-US0204/7
Other:
- moved on the sheet: U1
Changed lines of the file:
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@@
 <part name="FRAME1" library="frames" deviceset="FRAME_B_L" device=""/>
 <part name="U1" library="nocLock" deviceset="ATMEGA328" device=""/>
-<part name="IC1" library="v-reg" deviceset="78XXL" device=""/>
 <part name="FRAME3" library="frames" deviceset="DINA-DOC" device=""/>
+<part name="L1" library="rcl" deviceset="L-US" device="0204/7" value="100uH"/>
+<part name="C1" library="rcl" deviceset="C-US" device="C0805K" value="100nF"/>
+<part name="C2" library="rcl" deviceset="C-US" device="C0805K"/>
+<part name="C3" library="rcl" deviceset="C-US" device="C0805K"/>
+<part name="C4" library="rcl" deviceset="C-US" device="C0805K"/>
+<part name="C5" library="rcl" deviceset="C-US" device="C0805K"/>
+<part name="SUPPLY1" library="supply2" deviceset="GND" device=""/>
+<part name="SUPPLY2" library="supply2" deviceset="GND" device=""/>
+<part name="SUPPLY3" library="supply2" deviceset="GND" device=""/>
+<part name="SUPPLY4" library="supply2" deviceset="GND" device=""/>
+<part name="SUPPLY5" library="supply2" deviceset="GND" device=""/>
+<part name="SUPPLY6" library="supply2" deviceset="GND" device=""/>
+<part name="SUPPLY7" library="supply2" deviceset="GND" device=""/>
 </parts>
 <sheets>
@@
 <instance part="FRAME1" gate="G$1" x="66.04" y="30.48"/>
 <instance part="FRAME1" gate="G$2" x="391.16" y="30.48"/>
-<instance part="U1" gate="G$1" x="281.94" y="180.34"/>
-<instance part="IC1" gate="A" x="190.5" y="246.38"/>
+<instance part="U1" gate="G$1" x="193.04" y="195.58"/>
 <instance part="FRAME3" gate="G$1" x="406.4" y="259.08"/>
+<instance part="L1" gate="G$1" x="137.16" y="198.12"/>
+<instance part="C1" gate="G$1" x="137.16" y="177.8"/>
+<instance part="C2" gate="G$1" x="228.6" y="243.84"/>
+<instance part="C3" gate="G$1" x="218.44" y="243.84"/>
+<instance part="C4" gate="G$1" x="208.28" y="243.84"/>
+<instance part="C5" gate="G$1" x="200.66" y="241.3"/>
+<instance part="SUPPLY1" gate="GND" x="137.16" y="167.64"/>
+<instance part="SUPPLY2" gate="GND" x="127" y="162.56"/>
+<instance part="SUPPLY3" gate="GND" x="114.3" y="162.56"/>
+<instance part="SUPPLY4" gate="GND" x="109.22" y="160.02"/>
+<instance part="SUPPLY5" gate="GND" x="99.06" y="165.1"/>
+<instance part="SUPPLY6" gate="GND" x="109.22" y="170.18"/>
+<instance part="SUPPLY7" gate="GND" x="124.46" y="165.1"/>
 </instances>
 <busses>
