File: 411 Project/nocLock/100-Schematics/nocLock_proj/noclock_rev2.brd (EAGLE design)
At the start: 100 x 80 mm, 41 parts, among them J1 ICSP, J2 640455-2, J3 5BC-3-CA-F, Q1 DMN63D8LDW-7, Q3 DMG1012UW-7, U1 ATMEGA88A, U2 4584D, U3 MCP1802

Commit message: Started Board Layout
Parts:
- removed C12: (no value), rcl:C0805
- removed D5, D6: (no value), zetex:SOT-23
- removed FRAME2: (no value), nocLock_temp:DINA-DOC
- removed R12: (no value), rcl:R0805
- added J4, J5, J6, J7: 640455-2, nocLock_temp:2-PIN_CONNECTOR
- added R1210K: 10K, rcl:R0805
- added TP1: TPB1,27, testpad:B1,27
- added U$1: PMEG2005CT,215, nocLock_temp:SOT-23
- C7: value (none) -> 1uF
- J2: device nocLock_temp_Rev2:2-PIN_CONNECTOR -> nocLock_temp:2-PIN_CONNECTOR
- moved R2 180.2 mm to (88.9, 31.8), turned to 90 degrees
- moved J1 157.0 mm to (76.2, 25.4)
- moved R13 144.6 mm to (67.3, 55.9), turned to 180 degrees
- moved D1 136.5 mm to (82.5, 30.5), turned to 270 degrees
- moved R10 134.2 mm to (55.9, 26.7), turned to 90 degrees
- moved Q1 133.8 mm to (43.2, 19.1), turned to 90 degrees
- moved C5 128.9 mm to (72.4, 35.6), turned to 90 degrees
- moved D2 127.4 mm to (59.7, 14.0), turned to 270 degrees
- moved R8 116.6 mm to (49.5, 22.9), turned to 90 degrees
- moved R1 114.3 mm to (33.0, 72.4), turned to 90 degrees
- moved R6 114.3 mm to (67.3, 17.8), turned to 270 degrees
- moved D3 110.5 mm to (67.3, 63.5), turned to 270 degrees
- moved C7 109.3 mm to (22.9, 41.9), turned to 180 degrees
- moved C6 107.6 mm to (73.7, 19.1), turned to 90 degrees
- moved Q3 106.2 mm to (59.7, 21.6), turned to 180 degrees
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Connections:
- removed net AREF: U1.20
- removed net GND1: S2.1, S2.2
- removed net N$16: S2.3, S2.4
- new net N$1: J3.1, Q1.D1
- new net N$5: J3.3, Q1.D2
- new net N$6: TP1.TP, U1.20
- net +5V: now also J3.2, R1210K.1; no longer C12.1, R12.1, U3.4
- net +9V: now also J6.1, U$1.2; no longer D5.1, D6.1
- net GND: now also J2.2, J4.2, J5.2, J7.2, S2.1, S2.2; no longer C12.2
- net KNOCK_SENSE: now also J7.1
- net N$10: now also J6.2
- net N$15: now also S2.3, S2.4
- net N$19: now also R1210K.2; no longer R12.2
- net N$3: now also J2.1
- net N$4: now also J5.1, U$1.3; no longer D5.3
- net RESET1: now also J4.1, U$1.1; no longer D6.3
Routing:
- net GND: track 0.00 -> 386.3 mm, vias 0 -> 10
- net +5V: track 0.00 -> 235.7 mm, vias 0 -> 2
- net N$15: track 0.00 -> 115.4 mm, vias 0 -> 5
- net +9V: track 0.00 -> 67.9 mm, vias 0 -> 2
- net N$3: track 0.00 -> 67.3 mm
- net RESET: track 0.00 -> 55.7 mm, vias 0 -> 2
- net N$19: track 0.00 -> 54.1 mm, vias 0 -> 2
- net MOSI: track 0.00 -> 45.2 mm, vias 0 -> 3
- net N$7: track 0.00 -> 40.7 mm, vias 0 -> 2
- net KNOCK_SENSE: track 0.00 -> 34.0 mm
- net MISO: track 0.00 -> 30.1 mm, vias 0 -> 2
- net UNLOCK: track 0.00 -> 26.8 mm, vias 0 -> 2
- net N$10: track 0.00 -> 25.8 mm
- net SCK: track 0.00 -> 25.3 mm, vias 0 -> 2
- net PROGRAM: track 0.00 -> 15.4 mm, vias 0 -> 2
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Other:
- board size 100 x 80 mm -> 86.4 x 80 mm
