File: 411 Project/nocLock/100-Schematics/nocLock_proj/noclock_rev2.sch (EAGLE design)
At the start: 41 parts, among them J1 ICSP, J2 640455-2, J3 5BC-3-CA-F, Q1 DMN63D8LDW-7, Q3 DMG1012UW-7, U1 ATMEGA88A, U2 4584D, U3 MCP1802

Commit message: added connectors
Parts:
- removed C12: (no value), rcl:C-EUC0805
- added J4, J5, J6, J7: 640455-2, nocLock_temp:640455-2
- J2: device nocLock_temp_Rev2:640455-2 -> nocLock_temp:640455-2
Connections:
- new net N$1: J3.1, Q1A.D
- new net N$5: J3.3, Q1B.D
- net +5V: now also J3.2; no longer C12.1, U2P.VDD
- net +9V: now also J6.1
- net GND: now also J2.2, J4.2, J5.2, J7.2; no longer C12.2, U2P.VSS
- net KNOCK_SENSE: now also J7.1
- net N$10: now also J6.2
- net N$3: now also J2.1
- net N$4: now also J5.1
- net RESET1: now also J4.1
Other:
- moved on the sheet: J2, J3, Q1A, R3, R4

Commit message: updated schematic
Parts:
- added TP1: TPB1,27, testpad:TPB1,27
- C7: value (none) -> 1uF
- R1210K: value (none) -> 10K
- renumbered R12 to R1210K
Connections:
- removed net GND1: S2.1.1, S2.1.2
- removed net N$16: S2.2.1, S2.2.2
- new net N$6: TP1.TP, U1.AREF
- net +5V: now also U2P.VDD; no longer U3.NC
- net GND: now also S2.1.1, S2.1.2, U2P.VSS
- net N$15: now also S2.2.1, S2.2.2
Other:
- moved on the sheet: C11
Changed lines of the file:
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@@
 <setting verticaltext="up"/>
 </settings>
-<grid distance="0.1" unitdist="inch" unit="inch" style="lines" multiple="1" display="yes" altdistance="0.01" altunitdist="inch" altunit="inch"/>
+<grid distance="0.1" unitdist="inch" unit="inch" style="lines" multiple="1" display="no" altdistance="0.01" altunitdist="inch" altunit="inch"/>
 <layers>
 <layer number="1" name="Top" color="4" fill="1" visible="no" active="no"/>
@@
 <part name="SUPPLY2" library="supply2" deviceset="GND" device=""/>
 <part name="SUPPLY3" library="supply2" deviceset="GND" device=""/>
-<part name="C7" library="rcl" deviceset="C-EU" device="C0805"/>
-<part name="R12" library="rcl" deviceset="R-US_" device="R0805"/>
+<part name="C7" library="rcl" deviceset="C-EU" device="C0805" value="1uF"/>
+<part name="R1210K" library="rcl" deviceset="R-US_" device="R0805" value="10K"/>
 <part name="SUPPLY6" library="supply2" deviceset="GND" device=""/>
 <part name="SUPPLY7" library="supply2" deviceset="GND" device=""/>
@@
 <part name="J6" library="nocLock_temp" deviceset="640455-2" device=""/>
 <part name="J7" library="nocLock_temp" deviceset="640455-2" device=""/>
+<part name="SUPPLY17" library="supply2" deviceset="GND" device=""/>
+<part name="TP1" library="testpad" deviceset="TP" device="B1,27"/>
 </parts>
 <sheets>
@@
 <instance part="SUPPLY3" gate="GND" x="436.88" y="109.22"/>
 <instance part="C7" gate="G$1" x="99.06" y="266.7"/>
-<instance part="R12" gate="G$1" x="99.06" y="281.94" rot="R270"/>
+<instance part="R1210K" gate="G$1" x="99.06" y="281.94" rot="R270"/>
 <instance part="SUPPLY6" gate="GND" x="210.82" y="165.1"/>
 <instance part="SUPPLY7" gate="GND" x="213.36" y="190.5"/>
@@
 <instance part="SUPPLY5" gate="GND" x="127" y="45.72"/>
 <instance part="C10" gate="G$1" x="152.4" y="78.74"/>
-<instance part="C11" gate="G$1" x="185.42" y="78.74"/>
+<instance part="C11" gate="G$1" x="187.96" y="83.82"/>
 <instance part="SUPPLY15" gate="GND" x="170.18" y="55.88"/>
 <instance part="P+8" gate="1" x="198.12" y="121.92"/>
@@
 <instance part="J6" gate="G$1" x="449.58" y="187.96"/>
 <instance part="J7" gate="G$1" x="378.46" y="276.86"/>
+<instance part="U2" gate="P" x="198.12" y="83.82"/>
+<instance part="SUPPLY17" gate="GND" x="198.12" y="58.42"/>
+<instance part="TP1" gate="G$1" x="205.74" y="154.94" rot="R90"/>
 </instances>
 <busses>
@@
 <pinref part="C8" gate="G$1" pin="2"/>
 <pinref part="SUPPLY9" gate="GND" pin="GND"/>
-<wire x1="101.6" y1="152.4" x2="101.6" y2="144.78" width="0.1524" layer="91"/>
+<wire x1="101.6" y1="152.4" x2="101.6" y2="147.32" width="0.1524" layer="91"/>
+<pinref part="S2" gate="G$1" pin="1.1"/>
+<pinref part="S2" gate="G$1" pin="1.2"/>
+<wire x1="101.6" y1="147.32" x2="101.6" y2="144.78" width="0.1524" layer="91"/>
+<wire x1="86.36" y1="147.32" x2="88.9" y2="147.32" width="0.1524" layer="91"/>
+<wire x1="88.9" y1="147.32" x2="101.6" y2="147.32" width="0.1524" layer="91"/>
+<junction x="88.9" y="147.32"/>
+<junction x="101.6" y="147.32"/>
 </segment>
 <segment>
@@
 <segment>
 <pinref part="C11" gate="G$1" pin="2"/>
-<wire x1="185.42" y1="73.66" x2="185.42" y2="68.58" width="0.1524" layer="91"/>
-<wire x1="185.42" y1="68.58" x2="170.18" y2="68.58" width="0.1524" layer="91"/>
+<wire x1="187.96" y1="78.74" x2="187.96" y2="68.58" width="0.1524" layer="91"/>
+<wire x1="187.96" y1="68.58" x2="170.18" y2="68.58" width="0.1524" layer="91"/>
 <wire x1="170.18" y1="68.58" x2="170.18" y2="58.42" width="0.1524" layer="91"/>
 <pinref part="SUPPLY15" gate="GND" pin="GND"/>
@@
 <wire x1="210.82" y1="167.64" x2="210.82" y2="170.18" width="0.1524" layer="91"/>
 <junction x="210.82" y="170.18"/>
+</segment>
+<segment>
+<pinref part="U2" gate="P" pin="VSS"/>
+<pinref part="SUPPLY17" gate="GND" pin="GND"/>
+<wire x1="198.12" y1="60.96" x2="198.12" y2="76.2" width="0.1524" layer="91"/>
 </segment>
 </net>
@@
 </segment>
 <segment>
-<pinref part="R12" gate="G$1" pin="1"/>
+<pinref part="R1210K" gate="G$1" pin="1"/>
 <pinref part="P+4" gate="1" pin="+5V"/>
 <wire x1="99.06" y1="287.02" x2="99.06" y2="292.1" width="0.1524" layer="91"/>
@@
 <segment>
 <pinref part="U3" gate="G$1" pin="VOUT"/>
+<wire x1="185.42" y1="101.6" x2="187.96" y2="101.6" width="0.1524" layer="91"/>
+<wire x1="187.96" y1="101.6" x2="198.12" y2="101.6" width="0.1524" layer="91"/>
+<wire x1="198.12" y1="101.6" x2="198.12" y2="119.38" width="0.1524" layer="91"/>
+<pinref part="P+8" gate="1" pin="+5V"/>
+<pinref part="U2" gate="P" pin="VDD"/>
+<wire x1="198.12" y1="101.6" x2="198.12" y2="91.44" width="0.1524" layer="91"/>
+<junction x="198.12" y="101.6"/>
 <pinref part="C11" gate="G$1" pin="1"/>
-<wire x1="185.42" y1="81.28" x2="185.42" y2="86.36" width="0.1524" layer="91"/>
-<wire x1="185.42" y1="86.36" x2="185.42" y2="101.6" width="0.1524" layer="91"/>
-<wire x1="185.42" y1="101.6" x2="198.12" y2="101.6" width="0.1524" layer="91"/>
-<wire x1="198.12" y1="101.6" x2="198.12" y2="119.38" width="0.1524" layer="91"/>
-<junction x="185.42" y="101.6"/>
-<pinref part="U3" gate="G$1" pin="NC"/>
-<junction x="185.42" y="86.36"/>
-<pinref part="P+8" gate="1" pin="+5V"/>
+<wire x1="187.96" y1="86.36" x2="187.96" y2="101.6" width="0.1524" layer="91"/>
+<junction x="187.96" y="101.6"/>
 </segment>
 <segment>
@@
 <net name="N$15" class="0">
 <segment>
+<wire x1="119.38" y1="162.56" x2="101.6" y2="162.56" width="0.1524" layer="91"/>
+<pinref part="U2" gate="B" pin="I"/>
+<pinref part="S2" gate="G$1" pin="2.2"/>
+<pinref part="S2" gate="G$1" pin="2.1"/>
+<wire x1="88.9" y1="160.02" x2="86.36" y2="160.02" width="0.1524" layer="91"/>
+<wire x1="86.36" y1="162.56" x2="86.36" y2="160.02" width="0.1524" layer="91"/>
+<junction x="86.36" y="160.02"/>
+<wire x1="86.36" y1="162.56" x2="101.6" y2="162.56" width="0.1524" layer="91"/>
+<pinref part="R5" gate="G$1" pin="2"/>
 <pinref part="C8" gate="G$1" pin="1"/>
-<pinref part="R5" gate="G$1" pin="2"/>
 <wire x1="101.6" y1="160.02" x2="101.6" y2="162.56" width="0.1524" layer="91"/>
+<junction x="101.6" y="162.56"/>
 <wire x1="101.6" y1="162.56" x2="101.6" y2="165.1" width="0.1524" layer="91"/>
-<wire x1="119.38" y1="162.56" x2="101.6" y2="162.56" width="0.1524" layer="91"/>
-<junction x="101.6" y="162.56"/>
-<pinref part="U2" gate="B" pin="I"/>
 </segment>
 </net>
@@
 <junction x="83.82" y="271.78"/>
 <pinref part="C7" gate="G$1" pin="1"/>
-<pinref part="R12" gate="G$1" pin="2"/>
+<pinref part="R1210K" gate="G$1" pin="2"/>
 <wire x1="99.06" y1="269.24" x2="99.06" y2="274.32" width="0.1524" layer="91"/>
 <wire x1="99.06" y1="274.32" x2="99.06" y2="276.86" width="0.1524" layer="91"/>
@@
 <pinref part="U2" gate="C" pin="I"/>
 <wire x1="139.7" y1="162.56" x2="142.24" y2="162.56" width="0.1524" layer="91"/>
-</segment>
-</net>
-<net name="GND1" class="0">
-<segment>
-<pinref part="S2" gate="G$1" pin="1.1"/>
-<pinref part="S2" gate="G$1" pin="1.2"/>
-<wire x1="86.36" y1="147.32" x2="88.9" y2="147.32" width="0.1524" layer="91"/>
-<wire x1="88.9" y1="147.32" x2="101.6" y2="147.32" width="0.1524" layer="91"/>
-<junction x="88.9" y="147.32"/>
-</segment>
-</net>
-<net name="N$16" class="0">
-<segment>
-<pinref part="S2" gate="G$1" pin="2.2"/>
-<pinref part="S2" gate="G$1" pin="2.1"/>
-<wire x1="88.9" y1="160.02" x2="86.36" y2="160.02" width="0.1524" layer="91"/>
-<wire x1="86.36" y1="162.56" x2="86.36" y2="160.02" width="0.1524" layer="91"/>
-<junction x="86.36" y="160.02"/>
-<wire x1="86.36" y1="162.56" x2="101.6" y2="162.56" width="0.1524" layer="91"/>
 </segment>
 </net>
@@
 </segment>
 </net>
+<net name="N$6" class="0">
+<segment>
+<pinref part="U1" gate="G$1" pin="AREF"/>
+<wire x1="231.14" y1="182.88" x2="226.06" y2="182.88" width="0.1524" layer="91"/>
+<pinref part="TP1" gate="G$1" pin="TP"/>
+<wire x1="208.28" y1="154.94" x2="226.06" y2="154.94" width="0.1524" layer="91"/>
+<wire x1="226.06" y1="154.94" x2="226.06" y2="182.88" width="0.1524" layer="91"/>
+</segment>
+</net>

Commit message: Started Board Layout
Parts:
- removed D5, D6: (no value), zetex:VAR2SOT23
- removed FRAME2: (no value), nocLock_temp:DINA-DOC
- added U$1: PMEG2005CT,215, nocLock_temp:PMEG2005CT,215
Connections:
- net +9V: now also U$1.C; no longer D5.C, D6.C
- net N$4: now also U$1.A1; no longer D5.A
- net RESET1: now also U$1.A2; no longer D6.A
Other:
- note removed: "10/23/14"
- note removed: "Cameron Tribe"
- note removed: "Jaime Rodriguez"
Changed lines of the file:
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@@
 <part name="SUPPLY15" library="supply2" deviceset="GND" device=""/>
 <part name="P+8" library="supply1" deviceset="+5V" device=""/>
-<part name="FRAME2" library="nocLock_temp" deviceset="DINA-DOC" device=""/>
 <part name="R3" library="rcl" deviceset="R-US_" device="R0805" value="1k"/>
 <part name="R4" library="rcl" deviceset="R-US_" device="R0805" value="10K"/>
@@
 <part name="SUPPLY14" library="supply2" deviceset="GND" device=""/>
 <part name="U$2" library="supply1" deviceset="+9V" device=""/>
-<part name="D5" library="zetex" deviceset="VAR2SOT23" device=""/>
-<part name="D6" library="zetex" deviceset="VAR2SOT23" device=""/>
 <part name="U$3" library="supply1" deviceset="+9V" device=""/>
 <part name="SUPPLY12" library="supply2" deviceset="GND" device=""/>
@@
 <part name="SUPPLY17" library="supply2" deviceset="GND" device=""/>
 <part name="TP1" library="testpad" deviceset="TP" device="B1,27"/>
+<part name="U$1" library="nocLock_temp" deviceset="PMEG2005CT,215" device=""/>
 </parts>
 <sheets>
@@
 <wire x1="266.7" y1="246.38" x2="187.96" y2="246.38" width="0.1524" layer="97"/>
 <text x="190.5" y="294.64" size="1.778" layer="97">ICSP</text>
-<text x="462.28" y="292.1" size="1.778" layer="94">Cameron Tribe</text>
-<text x="462.28" y="287.02" size="1.778" layer="94">Jaime Rodriguez</text>
-<text x="452.12" y="287.02" size="1.27" layer="94" distance="51">10/23/14</text>
 <wire x1="73.66" y1="241.3" x2="73.66" y2="187.96" width="0.1524" layer="97"/>
 <wire x1="73.66" y1="187.96" x2="139.7" y2="187.96" width="0.1524" layer="97"/>
@@
 <instance part="SUPPLY15" gate="GND" x="170.18" y="55.88"/>
 <instance part="P+8" gate="1" x="198.12" y="121.92"/>
-<instance part="FRAME2" gate="G$1" x="407.4414" y="259.8928"/>
 <instance part="R3" gate="G$1" x="314.96" y="93.98" smashed="yes" rot="R90">
 <attribute name="NAME" x="321.31" y="97.5614" size="1.778" layer="95" rot="R180"/>
@@
 <instance part="SUPPLY14" gate="GND" x="228.6" y="132.08"/>
 <instance part="U$2" gate="G$1" x="152.4" y="121.92"/>
-<instance part="D5" gate="A" x="111.76" y="101.6"/>
-<instance part="D6" gate="A" x="127" y="93.98" rot="R90"/>
 <instance part="U$3" gate="G$1" x="436.88" y="215.9" smashed="yes">
 <attribute name="VALUE" x="444.5" y="215.9" size="1.778" layer="96" rot="R180"/>
@@
 <instance part="SUPPLY17" gate="GND" x="198.12" y="58.42"/>
 <instance part="TP1" gate="G$1" x="205.74" y="154.94" rot="R90"/>
+<instance part="U$1" gate="G$1" x="121.92" y="101.6"/>
 </instances>
 <busses>
@@
 <net name="RESET1" class="0">
 <segment>
-<wire x1="127" y1="91.44" x2="127" y2="73.66" width="0.1524" layer="91"/>
+<wire x1="127" y1="93.98" x2="127" y2="73.66" width="0.1524" layer="91"/>
 <wire x1="121.92" y1="73.66" x2="127" y2="73.66" width="0.1524" layer="91"/>
-<pinref part="D6" gate="A" pin="A"/>
 <pinref part="J4" gate="G$1" pin="1"/>
+<pinref part="U$1" gate="G$1" pin="A2"/>
 </segment>
 </net>
@@
 <net name="N$4" class="0">
 <segment>
-<pinref part="D5" gate="A" pin="A"/>
-<wire x1="93.98" y1="101.6" x2="109.22" y2="101.6" width="0.1524" layer="91"/>
+<wire x1="93.98" y1="101.6" x2="119.38" y2="101.6" width="0.1524" layer="91"/>
 <pinref part="J5" gate="G$1" pin="1"/>
+<pinref part="U$1" gate="G$1" pin="A1"/>
 </segment>
 </net>
@@
 <wire x1="152.4" y1="86.36" x2="152.4" y2="101.6" width="0.1524" layer="91"/>
 <wire x1="152.4" y1="101.6" x2="152.4" y2="119.38" width="0.1524" layer="91"/>
-<wire x1="127" y1="96.52" x2="127" y2="101.6" width="0.1524" layer="91"/>
-<wire x1="114.3" y1="101.6" x2="127" y2="101.6" width="0.1524" layer="91"/>
-<wire x1="127" y1="101.6" x2="152.4" y2="101.6" width="0.1524" layer="91"/>
-<junction x="127" y="101.6"/>
-<pinref part="D6" gate="A" pin="C"/>
-<pinref part="D5" gate="A" pin="C"/>
 <pinref part="U$2" gate="G$1" pin="+9V"/>
-</segment>
-<segment>
+<pinref part="U$1" gate="G$1" pin="C"/>
+<wire x1="129.54" y1="101.6" x2="152.4" y2="101.6" width="0.1524" layer="91"/>
+</segment>
+<segment>
