File: 411 Project/nocLock/100-Schematic/noclock_rev3.sch (EAGLE design)
At the start: 33 parts, among them Q1 DMG1012UW-7, Q2 DMG1012UW-7, Q3 DMG1012UW-7, U1 ATMEGA88A, U2 4584D

Commit message: updated library
Parts:
- removed L2: (no value), rcl:L-USL4532C
- removed LD1: (no value), led:DUOLED-RG-A
- removed Q2: DMG1012UW-7, nocLock_temp:DMG1012UW-7
- removed R7: (no value), rcl:R-US_R0805
- added C10, C11: 0.1uF, rcl:C-EUC0805
- added C12: (no value), rcl:C-EUC0805
- added D3: 5.1V, diode:ZENER-DIODESOT23
- added D5, D6: (no value), zetex:VAR2SOT23
- added FRAME2: (no value), nocLock_temp:DINA-DOC
- added J1: ICSP, nocLock_temp_Rev2:ICSP
- added J2: 640455-2, nocLock_temp_Rev2:640455-2
- added J3: 5BC-3-CA-F, nocLock_temp_Rev2:5BC-3-CA-F
- added R13: 1M, rcl:R-US_R0805
- added U3: MCP1802, nocLock_temp:MCP1802
- C6: value (none) -> 1000uF
- C8: value (none) -> 1uF
- C9: value 0.1uF -> 1uF
- Q1: value DMG1012UW-7 -> DMN63D8LDW-7; device nocLock_temp:DMG1012UW-7 -> nocLock_temp_Rev2:DMN63D8LDW-7
- R1, R2, R4: value (none) -> 10K
- R3: value (none) -> 1k
- R5: value (none) -> 10k
- R6: value 18 -> 10; device rcl:R-US_R0805 -> rcl:R-US_R2512
- R8: value 10k -> 1k
- R9: value 10k -> 10K
Connections:
- net N$13 renamed PROGRAM
- removed net N$1: Q1.G, R4.1, R9.1
- removed net N$14: R11.2, U1.PB1(PCINT1/OC1A)
- removed net N$17: R3.2, U1.PB2(PCINT2/SS/OC1B)
- removed net N$18: R4.2, U1.PB3(PCINT3/OC2A/MOSI)
- removed net N$20: U1.PC6(RESET/PCINT14), U2C.O
- removed net N$5: Q2.D, R1.1
- removed net N$6: Q2.G, R3.1, R8.1
- removed net N$8: L2.2, R6.2
- removed net VCC: D2.C, L2.1
- new net +9V: C10.1, D2.C, D5.C, D6.C, U3.SHDN, U3.VIN
- new net KNOCK_SENSE: D3.C, R13.1, U1.PC5(ADC5/SCL/PCINT13)
- new net MISO: J1.1, R8.2, U1.PB4(PCINT4/MISO)
- new net MOSI: J1.4, R3.2, U1.PB3(PCINT3/OC2A/MOSI)
- new net N$21: Q1A.G, R3.1, R4.2
- new net RESET: D1.A, J1.5, R2.2, U1.PC6(RESET/PCINT14), U2C.O
- new net RESET1: D6.A
- new net SCK: J1.3, U1.PB5(SCK/PCINT5)
- new net SOLENOID_CONTROL: R11.2, U1.PB2(PCINT2/SS/OC1B)
- new net UNLOCK: U1.PB1(PCINT1/OC1A), U2D.O
- net +5V: now also C11.1, C12.1, D1.C, J1.2, R1.1, R2.1, U3.NC, U3.VOUT; no longer C9.1, LD1.A
- net GND: now also C10.2, C11.2, C12.2, D3.A, J1.6, Q1A.S, Q1B.S, R13.2, R4.1, R9.1, U3.GND; no longer Q1.S, Q2.S, R8.2, R9.2
- net N$10: now also R6.2; no longer R6.1, R7.2
- net N$11: now also R6.1; no longer R7.1
- net N$2: now also Q1B.G, R8.1, R9.2; no longer LD1.CG, R1.2
- net N$3: now also C9.1, R1.2, U2D.I; no longer LD1.CR, R2.2
- net N$4: now also D5.A; no longer Q1.D, R2.1
Other:
- note added: "10/23/14"
- note added: "Cameron Tribe"
- note added: "ICSP"
- note added: "Jaime Rodriguez"
- note added: "Knock Sensor"
- note added: "Power Suppy"
- note added: "Reset Button"
- note added: "Unlock Button"
- note removed: "Solenoid"
- moved on the sheet: C1, C2, C3, C4, C5, C6, C7, C8, C9, D1, D2, L1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
