File: 411 Project/nocLock/100-Schematic/T02_noclock_rev3.sch (EAGLE design)
At the start: 46 parts, among them J1 ICSP, J3 5BC-3-CA-F, J4 640455-2, J5 640455-2, J6 640455-2, J7 640455-2, J8 640455-2, Q1 DMN63D8LDW-7, Q3 DMG1012UW-7, U1 ATMEGA88A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

Commit message: Updated Schematic and Library
added part numbers to all parts as attributes.
Parts:
- removed D1: GF1, diode:GF1
- removed S1: SKHMPSE010, switch:SKHMPSE010
- added R15, R16, R17: 100, rcl:R-US_R0805
- added TP1: TPTP19R, testpad:TPTP19R
- C1, C5: PARTNUM (none) -> CL21A475KOFNNNE
- C10, C11: value 0.1uF -> 1uF; PARTNUM (none) -> CL21B105KBFNNNE
- C12: value (none) -> 1uF; PARTNUM (none) -> CL21B105KBFNNNE
- C2, C3: PARTNUM (none) -> GRM155R61A104KA01D
- C4: value 100nF -> 0.1uF; PARTNUM (none) -> GRM155R61A104KA01D
- C6: device rcl:C-EUC0805 -> rcl:CPOL-US; PARTNUM (none) -> EKY-100ELL102MH20D
- C7, C8, C9: PARTNUM (none) -> CL21B105KBFNNNE
- D2: PARTNUM (none) -> S1J
- D3: PARTNUM (none) -> BZX84C4V7-TP
- D4: PARTNUM (none) -> PMEG2005CT,215
- J1: PARTNUM (none) -> PRPC012DAANRC
- J3: PARTNUM (none) -> 5BC-3-CA-F
- J4, J5, J6, J7, J8: PARTNUM (none) -> 640455-2
- L1: device rcl:L-USL4532C -> rcl:L-USL0805; PARTNUM (none) -> CE201210-10NJ
- Q1: PARTNUM (none) -> DMN63D8LDW-7
- Q3: PARTNUM (none) -> DMG1012UW-7
- R1, R10, R12, R2, R4, R5, R9: PARTNUM (none) -> ESR10EZPJ103
- R11, R3, R8: PARTNUM (none) -> MCR10ERTF1001
- R13: PARTNUM (none) -> RMCF0805JT1M00
- R14: PARTNUM (none) -> RMCF0805FT220R
- R6: PARTNUM (none) -> CRM2512-JW-100ELF
- R7: PARTNUM (none) -> MCR10ERTF3300
- U1: PARTNUM (none) -> ATMEGA88A-AUR
- U2: PARTNUM (none) -> 4584D
- U3: PARTNUM (none) -> MCP1802
Connections:
- removed net GND1: S2.1.1, S2.1.2
- removed net N$15: C8.1, R5.2, U2B.I
- new net AVCC: C4.1, C5.1, L1.1, U1.AVCC
- new net N$13: TP1.TP, U1.AREF
- new net N$14: R17.1, S2.2.1, S2.2.2
- new net N$17: J6.1, R16.1
- net +5V: now also L1.2; no longer D1.C, L1.1, U3.NC
- net GND: now also S2.1.1, S2.1.2, U2E.I, U2F.I; no longer S1.1.1, S1.1.2
- net N$10: now also C6.+; no longer C6.1
- net N$11: now also C6.-; no longer C6.2
- net N$16: now also C8.1, R17.2, R5.2, U2B.I; no longer S2.2.1, S2.2.2
- net N$19: now also R15.2; no longer S1.2.1, S1.2.2
- net N$3: now also R16.2; no longer J6.1
- net N$7: now also R15.1; no longer C4.1, C5.1, L1.2, U1.AVCC
- net RESET: no longer D1.A
Other:
- note added: "Button partnum"
- note added: "GPTS203211B"
- note added: "Green Drive"
- note added: "Red Drive"
- note added: "To piezo buzzer"
- note added: "Unused IC"
- moved on the sheet: C11, C7, C9, D2, J6, J7, L1, Q3, R1, R10, R11, R12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

Commit message: Submitted PCB Rev 3
Parts:
- removed FRAME2: (no value), nocLock_temp:DINA-DOC
- added S1: 2-1825910-7, nocLock_temp:2-1825910-7
- added TP10, TP2, TP3, TP4, TP5, TP6, TP7, TP8, TP9: TPTP19R, testpad:TPTP19R
- C6: device rcl:CPOL-US -> nocLock_temp:EKY-100ELL102MH20D; PARTNUM EKY-100ELL102MH20D -> (none)
- J1: device nocLock_temp_Rev2:ICSP -> nocLock_temp:ICSP; PARTNUM PRPC012DAANRC -> (none)
- L1: value 10nH -> CE201210-10NJ; device rcl:L-USL0805 -> nocLock_temp:CE201210-10NJ; PARTNUM CE201210-10NJ -> (none)
- S2: value SKHMPSE010 -> GPTS203211B; device switch:SKHMPSE010 -> nocLock_temp:GPTS203211B
Connections:
- net N$4 renamed 9V
- net RESET1 renamed BATT
- net +5V: now also TP5.TP, TP6.TP, TP7.TP
- net +9V: now also TP10.TP, TP8.TP, TP9.TP
- net GND: now also S1.1, S1.2, S2.1, S2.2, TP2.TP, TP3.TP, TP4.TP; no longer S2.1.1, S2.1.2
- net N$14: now also S2.3, S2.4; no longer S2.2.1, S2.2.2
- net N$7: now also S1.3, S1.4
Other:
- note removed: "Button partnum"
- note removed: "GPTS203211B"
- moved on the sheet: L1, S2
