File: 411 Project/nocLock/100-Schematic/T02_noclock_rev3.brd (EAGLE design)
At the start: 81.3 x 81.3 mm, 57 parts, among them J1 ICSP, J3 5BC-3-CA-F, J4 640455-2, J5 640455-2, J6 640455-2, J7 640455-2, J8 640455-2, Q1 DMN63D8LDW-7, Q3 DMG1012UW-7, U1 ATMEGA88A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

Commit message: Revised PCB layout.
Some work still needs to be done. Figure out a 5V power place rather
than a single trace to all things 5V.
Parts:
- moved TP5 21.6 mm to (33.0, 11.4)
- moved Q3 8.85 mm to (62.6, 34.1)
- moved D2 7.97 mm to (62.5, 21.5), flipped to the bottom, turned to 315 degrees
- moved C6 7.84 mm to (69.1, 34.2), turned to 180 degrees
- moved R10 7.55 mm to (71.6, 41.2), turned to 180 degrees
- moved TP1 5.81 mm to (56.4, 31.5)
- moved R6 5.29 mm to (69.1, 26.5)
- moved TP7 5.09 mm to (52.1, 59.4)
- moved R11 2.53 mm to (66.4, 41.2), turned to 180 degrees
Routing:
- net GND: track 411.0 -> 375.6 mm, vias 21 -> 19
- net +5V: track 239.5 -> 217.4 mm
- net N$13: track 13.4 -> 6.53 mm, vias 2 -> 0
- net N$9: track 6.48 -> 12.6 mm
- net N$11: track 16.1 -> 12.0 mm
- net SCK: track 30.6 -> 32.3 mm
- net SOLENOID_CONTROL: track 20.8 -> 19.4 mm
- net N$10: track 23.7 -> 22.4 mm
Other:
- board text added: "ICSP"
