File: 411 Project/nocLock/100-Schematic/T02_noclock_rev4.sch (EAGLE design)
At the start: 55 parts, among them J1 ICSP, J2 640455-2, J3 5BC-3-CA-F, J4 640455-2, J5 640455-2, J6 640455-2, J7 640455-2, J8 ICSP, Q1 DMN63D8LDW-7, Q3 DMG1012UW-7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

Commit message: updated schematics
Parts:
- removed J8: ICSP, T02_nocLock:ICSP
Other:
- note added: "10/10/14"
- note added: "10/12/14"
- note added: "10/24/14"
- note added: "10/25/14"
- note added: "11/13/14"
- note added: "A-1"
- note added: "A-2"
- note added: "A-3"
- note added: "B-1"
- note added: "B-2"
- note added: "B-3"
- note added: "Power Suppy for U2"
- note added: "Test Points"
- moved on the sheet: C12, J3, Q1A, Q1B, R14, R3, R4, R7, R8, R9, TP1, TP10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
