File: 411 Project/nocLock/200-PCB FIles/nocLock_Rev1.sch (EAGLE design)
At the start: 48 parts, among them J1 ICSP, J3 5BC-3-CA-F, J4 640455-2, J5 640455-2, J6 640455-2, J7 640455-2, J8 640455-2, Q1 DMN63D8LDW-7, Q3 DMG1012UW-7, U1 ATMEGA88A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

Commit message: Submitted PCB Rev 3
Parts:
- removed FRAME2: (no value), nocLock_temp:DINA-DOC
- removed R15, R16, R17: 100, rcl:R-US_R0805
- added D1: GF1, diode:GF1
- added S1: SKHMPSE010, switch:SKHMPSE010
- C1, C5: PARTNUM CL21A475KOFNNNE -> (none)
- C10, C11: value 1uF -> 0.1uF; PARTNUM CL21B105KBFNNNE -> (none)
- C12, C7, C8, C9: PARTNUM CL21B105KBFNNNE -> (none)
- C2, C3: PARTNUM GRM155R61A104KA01D -> (none)
- C4: value 0.1uF -> 100nF; PARTNUM GRM155R61A104KA01D -> (none)
- C6: device rcl:CPOL-US -> rcl:C-EUC0805; PARTNUM EKY-100ELL102MH20D -> (none)
- D2: PARTNUM S1J -> (none)
- D3: PARTNUM BZX84C4V7-TP -> (none)
- D4: PARTNUM PMEG2005CT,215 -> (none)
- J1: PARTNUM PRPC012DAANRC -> (none)
- J3: PARTNUM 5BC-3-CA-F -> (none)
- J4, J5, J6, J7, J8: PARTNUM 640455-2 -> (none)
- L1: device rcl:L-USL0805 -> rcl:L-USL4532C; PARTNUM CE201210-10NJ -> (none)
- Q1: PARTNUM DMN63D8LDW-7 -> (none)
- Q3: PARTNUM DMG1012UW-7 -> (none)
- R1, R10, R12, R2, R4, R5, R9: PARTNUM ESR10EZPJ103 -> (none)
- R11, R3, R8: PARTNUM MCR10ERTF1001 -> (none)
- R13: PARTNUM RMCF0805JT1M00 -> (none)
- R14: PARTNUM RMCF0805FT220R -> (none)
- R6: PARTNUM CRM2512-JW-100ELF -> (none)
- R7: PARTNUM MCR10ERTF3300 -> (none)
- U1: PARTNUM ATMEGA88A-AUR -> (none)
- U2: PARTNUM 4584D -> (none)
- U3: PARTNUM MCP1802 -> (none)
Connections:
- removed net AVCC: C4.1, C5.1, L1.1, U1.AVCC
- removed net N$14: R17.1, S2.2.1, S2.2.2
- removed net N$17: J6.1, R16.1
- net +5V: now also D1.C, L1.1; no longer L1.2
- net GND: now also S1.1.1, S1.1.2; no longer U2E.I, U2F.I
- net N$10: now also C6.1; no longer C6.+
- net N$11: now also C6.2; no longer C6.-
- net N$16: now also S2.2.1, S2.2.2; no longer R17.2
- net N$19: now also S1.2.1, S1.2.2; no longer R15.2
- net N$3: now also J6.1; no longer R16.2
- net N$7: now also C4.1, C5.1, L1.2, U1.AVCC; no longer R15.1
- net RESET: now also D1.A
Other:
- note removed: "2-1825910-7"
- note removed: "Button partnum"
- note removed: "GPTS203211B"
- note removed: "Green Drive"
- note removed: "Red Drive"
- note removed: "To piezo buzzer"
- note removed: "Unused IC"
- moved on the sheet: C7, C9, D2, J6, J7, L1, Q3, R1, R10, R11, R12, R6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
